File: Calculator.kicad_sch (KiCad schematic)
At the start: 3 parts, among them U1 RP2040, U2 LM66100DCK

Commit message: progress
Parts:
- removed BT1: Battery, symbol Device:Battery
- removed U2: LM66100DCK, Package_TO_SOT_SMD:SOT-363_SC-70-6, symbol Power_Management:LM66100DCK
- added C1, C2: 15pF, symbol Device:C
- added R1: R, symbol Device:R
- added R2: 1K, symbol Device:R
- added R3: 10k, symbol Device:R
- added SW1: SW_Push, symbol Switch:SW_Push
- added X1: ABM8-272-T3, ABM8-272-T3_ABR, symbol 2024-08-24_00-45-33:ABM8-272-T3
Connections:
- net GND: now also U1.57 (GND), C1.1, C2.1, SW1.1, X1.2, X1.4
- net XIN: now reaches U1.20 (XIN)
- net XIN: now also C1.2, R1.1, X1.1
- net XOUT: now reaches U1.21 (XOUT)
- net XOUT: now also R1.2, R2.2
- net at U1.26 (RUN): now also R3.1, SW1.2
- new net: C2.2, R2.1, X1.3
Other:
- moved on the sheet: U1

Commit message: progress
Connections:
- net GND: now also U1.19 (TESTEN)
Other:
- moved on the sheet: C1, C2, R1, R2, X1

Commit message: progress
Parts:
- removed C1, C2: 15pF, symbol Device:C
- removed R1: R, symbol Device:R
- removed R2: 1K, symbol Device:R
- removed R3: 10k, symbol Device:R
- removed SW1: SW_Push, symbol Switch:SW_Push
- removed U1: RP2040, Package_DFN_QFN:QFN-56-1EP_7x7mm_P0.4mm_EP3.2x3.2mm, symbol MCU_RaspberryPi:RP2040
- removed X1: ABM8-272-T3, ABM8-272-T3_ABR, symbol 2024-08-24_00-45-33:ABM8-272-T3
Other:
- added sheet MCU (MCU.kicad_sch)
- added sheet USB (USB.kicad_sch)

Commit message: progress
Other:
- added sheet Buttons (buttons.kicad_sch)
Changed lines of the file:
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@@
+	)
+	(sheet
+		(at 19.05 38.1)
+		(size 12.7 5.08)
+		(fields_autoplaced yes)
+		(stroke
+			(width 0.1524)
+			(type solid)
+		)
+		(fill
+			(color 0 0 0 0.0000)
+		)
+		(property "Sheetname" "Buttons"
+			(at 19.05 37.3884 0)
+			(effects
+				(font
+					(size 1.27 1.27)
+				)
+				(justify left bottom)
+			)
+		)
+		(property "Sheetfile" "buttons.kicad_sch"
+			(at 19.05 43.7646 0)
+			(effects
+				(font
+					(size 1.27 1.27)
+				)
+				(justify left top)
+			)
+		)
+		(instances
+			(project "Calculator"
+				(path "/687c7ae9-6ddd-479c-b536-3da1a83a559b"
+					(page "4")
+				)
+			)
+		)
 	)
 	(sheet
