File: MCU.kicad_sch (KiCad schematic)
At the start: 8 parts, among them SW1 SW_Push, U1 RP2040, X1 ABM8-272-T3

Commit message: progress
Parts:
- C1, C2: footprint (none) -> Capacitor_SMD:C_0201_0603Metric
- R1: footprint (none) -> Connector_USB:USB_A_Stewart_SS-52100-001_Horizontal
- R2: footprint (none) -> Connector_USB:USB_A_Molex_105057_Vertical
- R3: footprint (none) -> Connector_USB:USB_A_Molex_48037-2200_Horizontal
- SW1: footprint (none) -> Button_Switch_SMD:SW_DIP_SPSTx01_Slide_6.7x4.1mm_W6.73mm_P2.54mm_LowProfile_JPin
- X1: footprint ABM8-272-T3_ABR -> custom:ABM8-272-T3_ABR
Changed lines of the file:
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@@
 			)
 		)
-		(property "Footprint" ""
+		(property "Footprint" "Connector_USB:USB_A_Molex_105057_Vertical"
 			(at 41.91 160.528 90)
 			(effects
@@
 			)
 		)
-		(property "Footprint" ""
+		(property "Footprint" "Connector_USB:USB_A_Stewart_SS-52100-001_Horizontal"
 			(at 29.718 29.21 90)
 			(effects
@@
 			)
 		)
-		(property "Footprint" ""
+		(property "Footprint" "Capacitor_SMD:C_0201_0603Metric"
 			(at 24.4348 173.99 0)
 			(effects
@@
 			)
 		)
-		(property "Footprint" ""
+		(property "Footprint" "Capacitor_SMD:C_0201_0603Metric"
 			(at 58.7248 173.99 0)
 			(effects
@@
 			)
 		)
-		(property "Footprint" ""
+		(property "Footprint" "Button_Switch_SMD:SW_DIP_SPSTx01_Slide_6.7x4.1mm_W6.73mm_P2.54mm_LowProfile_JPin"
 			(at 19.05 38.1 0)
 			(effects
@@
 			)
 		)
-		(property "Footprint" "ABM8-272-T3_ABR"
+		(property "Footprint" "custom:ABM8-272-T3_ABR"
 			(at 29.21 171.45 0)
 			(effects
@@
 			)
 		)
-		(property "Footprint" ""
+		(property "Footprint" "Connector_USB:USB_A_Molex_48037-2200_Horizontal"
 			(at 61.468 165.1 90)
 			(effects
