File: buttons.kicad_sch (KiCad schematic)
At the start: 48 parts, among them SW10 SW_MEC_5G, SW11 SW_MEC_5G, SW12 SW_MEC_5G, SW13 SW_MEC_5G, SW14 SW_MEC_5G, SW15 SW_MEC_5G, SW16 SW_MEC_5G, SW17 SW_MEC_5G, SW18 SW_MEC_5G, SW19 SW_MEC_5G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

Commit message: progress
Parts:
- added D25, D26, D27, D28, D29, D30, D31, D32, D33, D34, D35, D36, D37, D38, D39, D40, D41, D42, D43, D44, D45, D46, D47, D48: D, symbol Device:D
- added SW26, SW27, SW28, SW29, SW30, SW31, SW32, SW33, SW34, SW35, SW36, SW37, SW38, SW39, SW40, SW41, SW42, SW43, SW44, SW45, SW46, SW47, SW48, SW49: SW_MEC_5G, symbol Switch:SW_MEC_5G
Connections:
- net BTN_COL1: now also D25.1 (K), D26.1 (K), D27.1 (K), D28.1 (K), D29.1 (K), D30.1 (K)
- net BTN_COL2: now also D31.1 (K), D32.1 (K), D33.1 (K), D34.1 (K), D35.1 (K), D36.1 (K)
- net BTN_COL3: now also D37.1 (K), D38.1 (K), D39.1 (K), D40.1 (K), D41.1 (K), D42.1 (K)
- net BTN_COL4: now also D43.1 (K), D44.1 (K), D45.1 (K), D46.1 (K), D47.1 (K), D48.1 (K)
- net BTN_ROW1: now also SW26.1 (A), SW26.2 (A), SW32.1 (A), SW32.2 (A), SW38.1 (A), SW38.2 (A), SW44.1 (A), SW44.2 (A)
- net BTN_ROW2: now also SW27.1 (A), SW27.2 (A), SW33.1 (A), SW33.2 (A), SW39.1 (A), SW39.2 (A), SW45.1 (A), SW45.2 (A)
- net BTN_ROW3: now also SW28.1 (A), SW28.2 (A), SW34.1 (A), SW34.2 (A), SW40.1 (A), SW40.2 (A), SW46.1 (A), SW46.2 (A)
- net BTN_ROW4: now also SW29.1 (A), SW29.2 (A), SW35.1 (A), SW35.2 (A), SW41.1 (A), SW41.2 (A), SW47.1 (A), SW47.2 (A)
- net BTN_ROW5: now also SW30.1 (A), SW30.2 (A), SW36.1 (A), SW36.2 (A), SW42.1 (A), SW42.2 (A), SW48.1 (A), SW48.2 (A)
- net BTN_ROW6: now also SW31.1 (A), SW31.2 (A), SW37.1 (A), SW37.2 (A), SW43.1 (A), SW43.2 (A), SW49.1 (A), SW49.2 (A)
- new net: D45.2 (A), SW46.3 (B), SW46.4 (B)
- new net: D27.2 (A), SW28.3 (B), SW28.4 (B)
- new net: D36.2 (A), SW37.3 (B), SW37.4 (B)
- new net: D25.2 (A), SW26.3 (B), SW26.4 (B)
- new net: D30.2 (A), SW31.3 (B), SW31.4 (B)
- new net: D42.2 (A), SW43.3 (B), SW43.4 (B)
- new net: D39.2 (A), SW40.3 (B), SW40.4 (B)
- new net: D29.2 (A), SW30.3 (B), SW30.4 (B)
- new net: D26.2 (A), SW27.3 (B), SW27.4 (B)
- new net: D47.2 (A), SW48.3 (B), SW48.4 (B)
- new net: D34.2 (A), SW35.3 (B), SW35.4 (B)
- new net: D31.2 (A), SW32.3 (B), SW32.4 (B)
- new net: D28.2 (A), SW29.3 (B), SW29.4 (B)
- new net: D37.2 (A), SW38.3 (B), SW38.4 (B)
- new net: D46.2 (A), SW47.3 (B), SW47.4 (B)
- new net: D33.2 (A), SW34.3 (B), SW34.4 (B)
- new net: D35.2 (A), SW36.3 (B), SW36.4 (B)
- new net: D32.2 (A), SW33.3 (B), SW33.4 (B)
- new net: D40.2 (A), SW41.3 (B), SW41.4 (B)
- new net: D44.2 (A), SW45.3 (B), SW45.4 (B)
- new net: D38.2 (A), SW39.3 (B), SW39.4 (B)
- new net: D48.2 (A), SW49.3 (B), SW49.4 (B)
- new net: D43.2 (A), SW44.3 (B), SW44.4 (B)
- new net: D41.2 (A), SW42.3 (B), SW42.4 (B)

Commit message: pcb
Parts:
- removed D25, D26, D27, D28, D29, D30, D31, D32, D33, D34, D35, D36, D37, D38, D39, D40, D41, D42, D43, D44, D45, D46, D47, D48: D, symbol Device:D
- removed SW26, SW27, SW28, SW29, SW30, SW31, SW32, SW33, SW34, SW35, SW36, SW37, SW38, SW39, SW40, SW41, SW42, SW43, SW44, SW45, SW46, SW47, SW48, SW49: SW_MEC_5G, symbol Switch:SW_MEC_5G
