File: buttons.kicad_sch (KiCad schematic)
At the start: 6 parts, among them SW2 SW_MEC_5G, SW3 SW_MEC_5G, SW4 SW_MEC_5G

Commit message: progress
Parts:
- added D4, D5, D6: D, symbol Device:D
- added SW5, SW6, SW7: SW_MEC_5G, symbol Switch:SW_MEC_5G
Connections:
- net BTN_ROW1: now also D1.1 (K), D4.1 (K); no longer D3.1 (K)
- net BTN_ROW2: now reaches D2.1 (K)
- net BTN_ROW2: now also D5.1 (K), SW5.1 (A), SW5.2 (A), SW6.1 (A), SW6.2 (A), SW7.1 (A), SW7.2 (A)
- new net: D5.2 (A), SW6.3 (B), SW6.4 (B)
- new net: D6.2 (A), SW7.3 (B), SW7.4 (B)
- new net: D4.2 (A), SW5.3 (B), SW5.4 (B)
- new net BTN_ROW3: D3.1 (K), D6.1 (K)

Commit message: progress
Parts:
- added D10, D11, D12, D7, D8, D9: D, symbol Device:D
- added SW10, SW11, SW12, SW13, SW8, SW9: SW_MEC_5G, symbol Switch:SW_MEC_5G
Connections:
- net BTN_ROW1: no longer D1.1 (K), D4.1 (K)
- net BTN_ROW2: no longer D2.1 (K), D5.1 (K)
- net BTN_ROW3: now also SW10.1 (A), SW10.2 (A), SW8.1 (A), SW8.2 (A), SW9.1 (A), SW9.2 (A); no longer D3.1 (K), D6.1 (K)
- new net: D9.2 (A), SW10.3 (B), SW10.4 (B)
- new net: D11.2 (A), SW12.3 (B), SW12.4 (B)
- new net: D8.2 (A), SW9.3 (B), SW9.4 (B)
- new net: D7.2 (A), SW8.3 (B), SW8.4 (B)
- new net: D10.2 (A), SW11.3 (B), SW11.4 (B)
- new net: D12.2 (A), SW13.3 (B), SW13.4 (B)
- new net BTN_COL1: D1.1 (K), D10.1 (K), D4.1 (K), D7.1 (K)
- new net BTN_COL2: D11.1 (K), D2.1 (K), D5.1 (K), D8.1 (K)
- new net BTN_COL3: D12.1 (K), D3.1 (K), D6.1 (K), D9.1 (K)
- new net BTN_ROW4: SW11.1 (A), SW11.2 (A), SW12.1 (A), SW12.2 (A), SW13.1 (A), SW13.2 (A)
Other:
- moved on the sheet: D1, D2, D3, D4, D5, D6, SW2, SW3, SW4, SW5, SW6, SW7

Commit message: progress
Parts:
- added D13, D14, D15, D16, D17, D18, D19, D20, D21, D22, D23, D24: D, symbol Device:D
- added SW14, SW15, SW16, SW17, SW18, SW19, SW20, SW21, SW22, SW23, SW24, SW25: SW_MEC_5G, symbol Switch:SW_MEC_5G
Connections:
- net BTN_COL1: now also D13.1 (K), D14.1 (K), D15.1 (K), D16.1 (K)
- net BTN_COL2: now also D17.1 (K), D18.1 (K), D19.1 (K), D20.1 (K)
- net BTN_COL3: now also D21.1 (K), D22.1 (K), D23.1 (K), D24.1 (K)
- net BTN_ROW1: now also SW14.1 (A), SW14.2 (A), SW18.1 (A), SW18.2 (A), SW22.1 (A), SW22.2 (A)
- net BTN_ROW2: now also SW15.1 (A), SW15.2 (A), SW19.1 (A), SW19.2 (A), SW23.1 (A), SW23.2 (A)
- net BTN_ROW3: now also SW16.1 (A), SW16.2 (A), SW20.1 (A), SW20.2 (A), SW24.1 (A), SW24.2 (A)
- net BTN_ROW4: now also SW17.1 (A), SW17.2 (A), SW21.1 (A), SW21.2 (A), SW25.1 (A), SW25.2 (A)
- new net: D16.2 (A), SW17.3 (B), SW17.4 (B)
- new net: D22.2 (A), SW23.3 (B), SW23.4 (B)
- new net: D17.2 (A), SW18.3 (B), SW18.4 (B)
- new net: D20.2 (A), SW21.3 (B), SW21.4 (B)
- new net: D13.2 (A), SW14.3 (B), SW14.4 (B)
- new net: D24.2 (A), SW25.3 (B), SW25.4 (B)
- new net: D15.2 (A), SW16.3 (B), SW16.4 (B)
- new net: D18.2 (A), SW19.3 (B), SW19.4 (B)
- new net: D19.2 (A), SW20.3 (B), SW20.4 (B)
- new net: D21.2 (A), SW22.3 (B), SW22.4 (B)
- new net: D23.2 (A), SW24.3 (B), SW24.4 (B)
- new net: D14.2 (A), SW15.3 (B), SW15.4 (B)

Commit message: progress
Connections:
- net BTN_COL1: now also D17.1 (K), D18.1 (K); no longer D13.1 (K), D14.1 (K), D15.1 (K), D16.1 (K)
- net BTN_COL2: no longer D17.1 (K), D18.1 (K)
- net BTN_COL3: no longer D23.1 (K), D24.1 (K)
- net BTN_ROW1: no longer SW18.1 (A), SW18.2 (A), SW22.1 (A), SW22.2 (A)
- net BTN_ROW2: no longer SW19.1 (A), SW19.2 (A), SW23.1 (A), SW23.2 (A)
- net BTN_ROW3: no longer SW20.1 (A), SW20.2 (A), SW24.1 (A), SW24.2 (A)
- net BTN_ROW4: no longer SW21.1 (A), SW21.2 (A), SW25.1 (A), SW25.2 (A)
- new net BTN_COL4: D13.1 (K), D14.1 (K), D15.1 (K), D16.1 (K), D23.1 (K), D24.1 (K)
- new net BTN_ROW5: SW18.1 (A), SW18.2 (A), SW20.1 (A), SW20.2 (A), SW22.1 (A), SW22.2 (A), SW24.1 (A), SW24.2 (A)
- new net BTN_ROW6: SW19.1 (A), SW19.2 (A), SW21.1 (A), SW21.2 (A), SW23.1 (A), SW23.2 (A), SW25.1 (A), SW25.2 (A)

Commit message: progress
Parts:
- D1, D10, D11, D12, D13, D14, D15, D16, D17, D18, D19, D2, D20, D21, D22, D23, D24, D3, D4, D5, D6, D7, D8, D9: footprint (none) -> Diode_SMD:D_0201_0603Metric
- SW10, SW11, SW12, SW13, SW14, SW15, SW16, SW17, SW18, SW19, SW2, SW20, SW21, SW22, SW23, SW24, SW25, SW3, SW4, SW5, SW6, SW7, SW8, SW9: footprint (none) -> Button_Switch_SMD:SW_DIP_SPSTx01_Slide_6.7x4.1mm_W6.73mm_P2.54mm_LowProfile_JPin
Changed lines of the file:
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@@
 			)
 		)
-		(property "Footprint" ""
+		(property "Footprint" "Button_Switch_SMD:SW_DIP_SPSTx01_Slide_6.7x4.1mm_W6.73mm_P2.54mm_LowProfile_JPin"
 			(at 120.65 86.36 0)
 			(effects
@@
 			)
 		)
-		(property "Footprint" ""
+		(property "Footprint" "Button_Switch_SMD:SW_DIP_SPSTx01_Slide_6.7x4.1mm_W6.73mm_P2.54mm_LowProfile_JPin"
 			(at 54.61 100.33 0)
 			(effects
@@
 			)
 		)
-		(property "Footprint" ""
+		(property "Footprint" "Diode_SMD:D_0201_0603Metric"
 			(at 85.09 35.56 0)
 			(effects
@@
 			)
 		)
-		(property "Footprint" ""
+		(property "Footprint" "Diode_SMD:D_0201_0603Metric"
 			(at 106.68 63.5 0)
 			(effects
@@
 			)
 		)
-		(property "Footprint" ""
+		(property "Footprint" "Button_Switch_SMD:SW_DIP_SPSTx01_Slide_6.7x4.1mm_W6.73mm_P2.54mm_LowProfile_JPin"
 			(at 120.65 30.48 0)
 			(effects
@@
 			)
 		)
-		(property "Footprint" ""
+		(property "Footprint" "Diode_SMD:D_0201_0603Metric"
 			(at 106.68 35.56 0)
 			(effects
@@
 			)
 		)
-		(property "Footprint" ""
+		(property "Footprint" "Diode_SMD:D_0201_0603Metric"
 			(at 85.09 77.47 0)
 			(effects
@@
 			)
 		)
-		(property "Footprint" ""
+		(property "Footprint" "Button_Switch_SMD:SW_DIP_SPSTx01_Slide_6.7x4.1mm_W6.73mm_P2.54mm_LowProfile_JPin"
 			(at 97.79 100.33 0)
 			(effects
@@
 			)
 		)
-		(property "Footprint" ""
+		(property "Footprint" "Diode_SMD:D_0201_0603Metric"
 			(at 63.5 91.44 0)
 			(effects
@@
 			)
 		)
-		(property "Footprint" ""
+		(property "Footprint" "Button_Switch_SMD:SW_DIP_SPSTx01_Slide_6.7x4.1mm_W6.73mm_P2.54mm_LowProfile_JPin"
 			(at 76.2 72.39 0)
 			(effects
@@
 			)
 		)
-		(property "Footprint" ""
+		(property "Footprint" "Diode_SMD:D_0201_0603Metric"
 			(at 129.54 105.41 0)
 			(effects
@@
 			)
 		)
-		(property "Footprint" ""
+		(property "Footprint" "Diode_SMD:D_0201_0603Metric"
 			(at 85.09 63.5 0)
 			(effects
@@
 			)
 		)
-		(property "Footprint" ""
+		(property "Footprint" "Diode_SMD:D_0201_0603Metric"
 			(at 63.5 35.56 0)
 			(effects
@@
 			)
 		)
-		(property "Footprint" ""
+		(property "Footprint" "Diode_SMD:D_0201_0603Metric"
 			(at 63.5 105.41 0)
 			(effects
@@
 			)
 		)
-		(property "Footprint" ""
+		(property "Footprint" "Button_Switch_SMD:SW_DIP_SPSTx01_Slide_6.7x4.1mm_W6.73mm_P2.54mm_LowProfile_JPin"
 			(at 120.65 58.42 0)
 			(effects
@@
 			)
 		)
-		(property "Footprint" ""
+		(property "Footprint" "Diode_SMD:D_0201_0603Metric"
 			(at 129.54 49.53 0)
 			(effects
@@
 			)
 		)
-		(property "Footprint" ""
+		(property "Footprint" "Diode_SMD:D_0201_0603Metric"
 			(at 106.68 105.41 0)
 			(effects
@@
 			)
 		)
-		(property "Footprint" ""
+		(property "Footprint" "Button_Switch_SMD:SW_DIP_SPSTx01_Slide_6.7x4.1mm_W6.73mm_P2.54mm_LowProfile_JPin"
 			(at 76.2 30.48 0)
 			(effects
@@
 			)
 		)
-		(property "Footprint" ""
+		(property "Footprint" "Diode_SMD:D_0201_0603Metric"
 			(at 129.54 63.5 0)
 			(effects
@@
 			)
 		)
-		(property "Footprint" ""
+		(property "Footprint" "Button_Switch_SMD:SW_DIP_SPSTx01_Slide_6.7x4.1mm_W6.73mm_P2.54mm_LowProfile_JPin"
 			(at 76.2 44.45 0)
 			(effects
@@
 			)
 		)
-		(property "Footprint" ""
+		(property "Footprint" "Button_Switch_SMD:SW_DIP_SPSTx01_Slide_6.7x4.1mm_W6.73mm_P2.54mm_LowProfile_JPin"
 			(at 97.79 86.36 0)
 			(effects
@@
 			)
 		)
-		(property "Footprint" ""
+		(property "Footprint" "Button_Switch_SMD:SW_DIP_SPSTx01_Slide_6.7x4.1mm_W6.73mm_P2.54mm_LowProfile_JPin"
 			(at 76.2 58.42 0)
 			(effects
@@
 			)
 		)
-		(property "Footprint" ""
+		(property "Footprint" "Button_Switch_SMD:SW_DIP_SPSTx01_Slide_6.7x4.1mm_W6.73mm_P2.54mm_LowProfile_JPin"
 			(at 97.79 44.45 0)
 			(effects
@@
 			)
 		)
-		(property "Footprint" ""
+		(property "Footprint" "Diode_SMD:D_0201_0603Metric"
 			(at 129.54 77.47 0)
 			(effects
@@
 			)
 		)
-		(property "Footprint" ""
+		(property "Footprint" "Button_Switch_SMD:SW_DIP_SPSTx01_Slide_6.7x4.1mm_W6.73mm_P2.54mm_LowProfile_JPin"
 			(at 54.61 86.36 0)
 			(effects
@@
 			)
 		)
-		(property "Footprint" ""
+		(property "Footprint" "Button_Switch_SMD:SW_DIP_SPSTx01_Slide_6.7x4.1mm_W6.73mm_P2.54mm_LowProfile_JPin"
 			(at 76.2 86.36 0)
 			(effects
@@
 			)
 		)
-		(property "Footprint" ""
+		(property "Footprint" "Diode_SMD:D_0201_0603Metric"
 			(at 106.68 49.53 0)
 			(effects
@@
 			)
 		)
-		(property "Footprint" ""
+		(property "Footprint" "Button_Switch_SMD:SW_DIP_SPSTx01_Slide_6.7x4.1mm_W6.73mm_P2.54mm_LowProfile_JPin"
 			(at 76.2 100.33 0)
 			(effects
@@
 			)
 		)
-		(property "Footprint" ""
+		(property "Footprint" "Diode_SMD:D_0201_0603Metric"
 			(at 129.54 91.44 0)
 			(effects
@@
 			)
 		)
-		(property "Footprint" ""
+		(property "Footprint" "Diode_SMD:D_0201_0603Metric"
 			(at 85.09 49.53 0)
 			(effects
@@
 			)
 		)
-		(property "Footprint" ""
+		(property "Footprint" "Diode_SMD:D_0201_0603Metric"
 			(at 63.5 49.53 0)
 			(effects
@@
 			)
 		)
-		(property "Footprint" ""
+		(property "Footprint" "Diode_SMD:D_0201_0603Metric"
 			(at 63.5 63.5 0)
 			(effects
@@
 			)
 		)
-		(property "Footprint" ""
+		(property "Footprint" "Diode_SMD:D_0201_0603Metric"
 			(at 63.5 77.47 0)
 			(effects
@@
 			)
 		)
-		(property "Footprint" ""
+		(property "Footprint" "Button_Switch_SMD:SW_DIP_SPSTx01_Slide_6.7x4.1mm_W6.73mm_P2.54mm_LowProfile_JPin"
 			(at 97.79 30.48 0)
 			(effects
@@
 			)
 		)
-		(property "Footprint" ""
+		(property "Footprint" "Button_Switch_SMD:SW_DIP_SPSTx01_Slide_6.7x4.1mm_W6.73mm_P2.54mm_LowProfile_JPin"
 			(at 97.79 58.42 0)
 			(effects
@@
 			)
 		)
-		(property "Footprint" ""
+		(property "Footprint" "Diode_SMD:D_0201_0603Metric"
 			(at 106.68 91.44 0)
 			(effects
@@
 			)
 		)
-		(property "Footprint" ""
+		(property "Footprint" "Button_Switch_SMD:SW_DIP_SPSTx01_Slide_6.7x4.1mm_W6.73mm_P2.54mm_LowProfile_JPin"
 			(at 54.61 72.39 0)
 			(effects
@@
 			)
 		)
-		(property "Footprint" ""
+		(property "Footprint" "Button_Switch_SMD:SW_DIP_SPSTx01_Slide_6.7x4.1mm_W6.73mm_P2.54mm_LowProfile_JPin"
 			(at 120.65 72.39 0)
 			(effects
@@
 			)
 		)
-		(property "Footprint" ""
+		(property "Footprint" "Button_Switch_SMD:SW_DIP_SPSTx01_Slide_6.7x4.1mm_W6.73mm_P2.54mm_LowProfile_JPin"
 			(at 54.61 30.48 0)
 			(effects
@@
 			)
 		)
-		(property "Footprint" ""
+		(property "Footprint" "Button_Switch_SMD:SW_DIP_SPSTx01_Slide_6.7x4.1mm_W6.73mm_P2.54mm_LowProfile_JPin"
 			(at 120.65 100.33 0)
 			(effects
@@
 			)
 		)
-		(property "Footprint" ""
+		(property "Footprint" "Diode_SMD:D_0201_0603Metric"
 			(at 85.09 105.41 0)
 			(effects
@@
 			)
 		)
-		(property "Footprint" ""
+		(property "Footprint" "Button_Switch_SMD:SW_DIP_SPSTx01_Slide_6.7x4.1mm_W6.73mm_P2.54mm_LowProfile_JPin"
 			(at 54.61 58.42 0)
 			(effects
@@
 			)
 		)
-		(property "Footprint" ""
+		(property "Footprint" "Button_Switch_SMD:SW_DIP_SPSTx01_Slide_6.7x4.1mm_W6.73mm_P2.54mm_LowProfile_JPin"
 			(at 120.65 44.45 0)
 			(effects
@@
 			)
 		)
-		(property "Footprint" ""
+		(property "Footprint" "Button_Switch_SMD:SW_DIP_SPSTx01_Slide_6.7x4.1mm_W6.73mm_P2.54mm_LowProfile_JPin"
 			(at 97.79 72.39 0)
 			(effects
@@
 			)
 		)
-		(property "Footprint" ""
+		(property "Footprint" "Diode_SMD:D_0201_0603Metric"
 			(at 85.09 91.44 0)
 			(effects
@@
 			)
 		)
-		(property "Footprint" ""
+		(property "Footprint" "Button_Switch_SMD:SW_DIP_SPSTx01_Slide_6.7x4.1mm_W6.73mm_P2.54mm_LowProfile_JPin"
 			(at 54.61 44.45 0)
 			(effects
@@
 			)
 		)
-		(property "Footprint" ""
+		(property "Footprint" "Diode_SMD:D_0201_0603Metric"
 			(at 106.68 77.47 0)
 			(effects
@@
 			)
 		)
-		(property "Footprint" ""
+		(property "Footprint" "Diode_SMD:D_0201_0603Metric"
 			(at 129.54 35.56 0)
 			(effects
