File: Calculator.kicad_pcb (KiCad board)
At the start: 2 copper layers, 2 parts, among them U1 RP2040, X1 ABM8-272-T3

Commit message: progress
Parts:
- added C1: 15pF, Capacitor_SMD:C_0201_0603Metric, F.Cu at (91.6, 104.1)
- added C2: 15pF, Capacitor_SMD:C_0201_0603Metric, F.Cu at (91.6, 105.9)
- added D1: D, Diode_SMD:D_0201_0603Metric, F.Cu at (63.0, 67.8)
- added D10: D, Diode_SMD:D_0201_0603Metric, F.Cu at (65.7, 73.1)
- added D11: D, Diode_SMD:D_0201_0603Metric, F.Cu at (65.7, 74.8)
- added D12: D, Diode_SMD:D_0201_0603Metric, F.Cu at (65.7, 76.6)
- added D13: D, Diode_SMD:D_0201_0603Metric, F.Cu at (68.4, 67.8)
- added D14: D, Diode_SMD:D_0201_0603Metric, F.Cu at (68.4, 69.6)
- added D15: D, Diode_SMD:D_0201_0603Metric, F.Cu at (68.4, 71.3)
- added D16: D, Diode_SMD:D_0201_0603Metric, F.Cu at (68.4, 73.1)
- added D17: D, Diode_SMD:D_0201_0603Metric, F.Cu at (68.4, 74.8)
- added D18: D, Diode_SMD:D_0201_0603Metric, F.Cu at (68.4, 76.6)
- added D19: D, Diode_SMD:D_0201_0603Metric, F.Cu at (71.1, 67.8)
- added D2: D, Diode_SMD:D_0201_0603Metric, F.Cu at (63.0, 69.6)
- added D20: D, Diode_SMD:D_0201_0603Metric, F.Cu at (71.1, 69.6)
- added D21: D, Diode_SMD:D_0201_0603Metric, F.Cu at (71.1, 71.3)
- added D22: D, Diode_SMD:D_0201_0603Metric, F.Cu at (71.1, 73.1)
- added D23: D, Diode_SMD:D_0201_0603Metric, F.Cu at (71.1, 74.8)
- added D24: D, Diode_SMD:D_0201_0603Metric, F.Cu at (71.1, 76.6)
- added D3: D, Diode_SMD:D_0201_0603Metric, F.Cu at (63.0, 71.3)
- added D4: D, Diode_SMD:D_0201_0603Metric, F.Cu at (63.0, 73.1)
- added D5: D, Diode_SMD:D_0201_0603Metric, F.Cu at (63.0, 74.8)
- added D6: D, Diode_SMD:D_0201_0603Metric, F.Cu at (63.0, 76.6)
- added D7: D, Diode_SMD:D_0201_0603Metric, F.Cu at (65.7, 67.8)
- added D8: D, Diode_SMD:D_0201_0603Metric, F.Cu at (65.7, 69.6)
- added D9: D, Diode_SMD:D_0201_0603Metric, F.Cu at (65.7, 71.3)
- added J1: USB_A, Connector_USB:USB_A_Receptacle_GCT_USB1046, F.Cu at (108.5, 92.6)
- added R1: 10k, Connector_USB:USB_A_Stewart_SS-52100-001_Horizontal, F.Cu at (67.2, 96.5)
- added R2: R, Connector_USB:USB_A_Molex_105057_Vertical, F.Cu at (85.0, 101.3)
- added R3: 1K, Connector_USB:USB_A_Molex_48037-2200_Horizontal, F.Cu at (48.6, 95.1)
- added SW1: SW_Push, Button_Switch_SMD:SW_DIP_SPSTx01_Slide_6.7x4.1mm_W6.73mm_P2.54mm_LowProfile_JPin, F.Cu at (85.1, 106.2)
- added SW10: SW_MEC_5G, Button_Switch_SMD:SW_DIP_SPSTx01_Slide_6.7x4.1mm_W6.73mm_P2.54mm_LowProfile_JPin, F.Cu at (77.2, 46.5)
- added SW11: SW_MEC_5G, Button_Switch_SMD:SW_DIP_SPSTx01_Slide_6.7x4.1mm_W6.73mm_P2.54mm_LowProfile_JPin, F.Cu at (77.2, 52.3)
- added SW12: SW_MEC_5G, Button_Switch_SMD:SW_DIP_SPSTx01_Slide_6.7x4.1mm_W6.73mm_P2.54mm_LowProfile_JPin, F.Cu at (77.2, 58.2)
- added SW13: SW_MEC_5G, Button_Switch_SMD:SW_DIP_SPSTx01_Slide_6.7x4.1mm_W6.73mm_P2.54mm_LowProfile_JPin, F.Cu at (77.2, 64.0)
- added SW14: SW_MEC_5G, Button_Switch_SMD:SW_DIP_SPSTx01_Slide_6.7x4.1mm_W6.73mm_P2.54mm_LowProfile_JPin, F.Cu at (87.7, 34.8)
- added SW15: SW_MEC_5G, Button_Switch_SMD:SW_DIP_SPSTx01_Slide_6.7x4.1mm_W6.73mm_P2.54mm_LowProfile_JPin, F.Cu at (87.7, 40.6)
- added SW16: SW_MEC_5G, Button_Switch_SMD:SW_DIP_SPSTx01_Slide_6.7x4.1mm_W6.73mm_P2.54mm_LowProfile_JPin, F.Cu at (87.7, 46.5)
- added SW17: SW_MEC_5G, Button_Switch_SMD:SW_DIP_SPSTx01_Slide_6.7x4.1mm_W6.73mm_P2.54mm_LowProfile_JPin, F.Cu at (87.7, 52.3)
- added SW18: SW_MEC_5G, Button_Switch_SMD:SW_DIP_SPSTx01_Slide_6.7x4.1mm_W6.73mm_P2.54mm_LowProfile_JPin, F.Cu at (87.7, 58.2)
- added SW19: SW_MEC_5G, Button_Switch_SMD:SW_DIP_SPSTx01_Slide_6.7x4.1mm_W6.73mm_P2.54mm_LowProfile_JPin, F.Cu at (87.7, 64.0)
- added SW2: SW_MEC_5G, Button_Switch_SMD:SW_DIP_SPSTx01_Slide_6.7x4.1mm_W6.73mm_P2.54mm_LowProfile_JPin, F.Cu at (66.8, 34.8)
- added SW20: SW_MEC_5G, Button_Switch_SMD:SW_DIP_SPSTx01_Slide_6.7x4.1mm_W6.73mm_P2.54mm_LowProfile_JPin, F.Cu at (98.1, 34.8)
- added SW21: SW_MEC_5G, Button_Switch_SMD:SW_DIP_SPSTx01_Slide_6.7x4.1mm_W6.73mm_P2.54mm_LowProfile_JPin, F.Cu at (98.1, 40.6)
- added SW22: SW_MEC_5G, Button_Switch_SMD:SW_DIP_SPSTx01_Slide_6.7x4.1mm_W6.73mm_P2.54mm_LowProfile_JPin, F.Cu at (98.1, 46.5)
- added SW23: SW_MEC_5G, Button_Switch_SMD:SW_DIP_SPSTx01_Slide_6.7x4.1mm_W6.73mm_P2.54mm_LowProfile_JPin, F.Cu at (98.1, 52.3)
- added SW24: SW_MEC_5G, Button_Switch_SMD:SW_DIP_SPSTx01_Slide_6.7x4.1mm_W6.73mm_P2.54mm_LowProfile_JPin, F.Cu at (98.1, 58.2)
- added SW25: SW_MEC_5G, Button_Switch_SMD:SW_DIP_SPSTx01_Slide_6.7x4.1mm_W6.73mm_P2.54mm_LowProfile_JPin, F.Cu at (98.1, 64.0)
- added SW3: SW_MEC_5G, Button_Switch_SMD:SW_DIP_SPSTx01_Slide_6.7x4.1mm_W6.73mm_P2.54mm_LowProfile_JPin, F.Cu at (66.8, 40.6)
- added SW4: SW_MEC_5G, Button_Switch_SMD:SW_DIP_SPSTx01_Slide_6.7x4.1mm_W6.73mm_P2.54mm_LowProfile_JPin, F.Cu at (66.8, 46.5)
- added SW5: SW_MEC_5G, Button_Switch_SMD:SW_DIP_SPSTx01_Slide_6.7x4.1mm_W6.73mm_P2.54mm_LowProfile_JPin, F.Cu at (66.8, 52.3)
- added SW6: SW_MEC_5G, Button_Switch_SMD:SW_DIP_SPSTx01_Slide_6.7x4.1mm_W6.73mm_P2.54mm_LowProfile_JPin, F.Cu at (66.8, 58.2)
- added SW7: SW_MEC_5G, Button_Switch_SMD:SW_DIP_SPSTx01_Slide_6.7x4.1mm_W6.73mm_P2.54mm_LowProfile_JPin, F.Cu at (66.8, 64.0)
- added SW8: SW_MEC_5G, Button_Switch_SMD:SW_DIP_SPSTx01_Slide_6.7x4.1mm_W6.73mm_P2.54mm_LowProfile_JPin, F.Cu at (77.2, 34.8)
- added SW9: SW_MEC_5G, Button_Switch_SMD:SW_DIP_SPSTx01_Slide_6.7x4.1mm_W6.73mm_P2.54mm_LowProfile_JPin, F.Cu at (77.2, 40.6)
- moved X1 58.0 mm to (139.5, 83.0)
- moved U1 55.9 mm to (133.3, 81.0)
